Commit message: Finished based setup.

File: schunk_lwa4p/urdf/robot.urdf.xacro (robot description, xacro)
@@ -1,15 +1 @@
-<?xml version="1.0"?>
-<robot xmlns:xacro="http://www.ros.org/wiki/xacro"
-       name="lwa4p" >
-  <!-- common stuff -->
-  <xacro:include filename="$(find schunk_description)/urdf/common.xacro" />
-  <xacro:include filename="$(find schunk_description)/urdf/materials.urdf.xacro" />
-  <!-- schunk lwa4p -->
-  <xacro:include filename="$(find schunk_description)/urdf/lwa4p/lwa4p.urdf.xacro" />
-  <!-- Used for fixing robot to Gazebo -->
-  <link name="world"/>
-  <!-- arm -->
-  <xacro:schunk_lwa4p name="arm" parent="world" has_podest="true">
-    <origin xyz="0 0 0.052" rpy="0 0 0" /> <!--slightly above gazebo plane-->
-  </xacro:schunk_lwa4p>
-</robot>
+schunk_lwa4p.urdf.xacro
